Commit message: Simplify Lambda RViz visualization

File: src/lambda07_bringup/urdf/lambda07.urdf.xacro (robot description, xacro)
@@ -26,31 +26,7 @@
       </visual>
     </link>
-    <link name="${robot_id}_x_link">
-      <visual>
-        <origin xyz="0.04 0 0" rpy="0 1.57079632679 0"/>
-        <geometry>
-          <cylinder radius="0.006" length="0.08"/>
-        </geometry>
-        <material name="lambda07_axis_x"/>
-      </visual>
-    </link>
-    <link name="${robot_id}_y_link">
-      <visual>
-        <origin xyz="0 0.04 0" rpy="1.57079632679 0 0"/>
-        <geometry>
-          <cylinder radius="0.006" length="0.08"/>
-        </geometry>
-        <material name="lambda07_axis_y"/>
-      </visual>
-    </link>
-    <link name="${robot_id}_z_link">
-      <visual>
-        <origin xyz="0 0 0.04" rpy="0 0 0"/>
-        <geometry>
-          <cylinder radius="0.006" length="0.08"/>
-        </geometry>
-        <material name="lambda07_axis_z"/>
-      </visual>
-    </link>
+    <link name="${robot_id}_x_link"/>
+    <link name="${robot_id}_y_link"/>
+    <link name="${robot_id}_z_link"/>
     <link name="${robot_id}_roll_link"/>
     <link name="${robot_id}_pitch_link"/>
@@ -64,14 +40,27 @@
         <material name="lambda07_ee_mat"/>
       </visual>
-    </link>
-    <link name="${robot_id}_virtual_clutch_link">
       <visual>
-        <origin xyz="0.025 0 0" rpy="0 1.57079632679 0"/>
+        <origin xyz="0.035 0 0" rpy="0 1.57079632679 0"/>
         <geometry>
-          <cylinder radius="0.004" length="0.05"/>
+          <cylinder radius="0.003" length="0.07"/>
         </geometry>
-        <material name="lambda07_ee_mat"/>
+        <material name="lambda07_axis_x"/>
+      </visual>
+      <visual>
+        <origin xyz="0 0.035 0" rpy="1.57079632679 0 0"/>
+        <geometry>
+          <cylinder radius="0.003" length="0.07"/>
+        </geometry>
+        <material name="lambda07_axis_y"/>
+      </visual>
+      <visual>
+        <origin xyz="0 0 0.035" rpy="0 0 0"/>
+        <geometry>
+          <cylinder radius="0.003" length="0.07"/>
+        </geometry>
+        <material name="lambda07_axis_z"/>
       </visual>
     </link>
+    <link name="${robot_id}_virtual_clutch_link"/>
     <joint name="${robot_id}_x" type="prismatic">
       <origin rpy="0 0 0" xyz="0 0 0"/>

Commit message: Fix Lambda wrist orientation mapping

File: src/lambda07_bringup/urdf/lambda07.urdf.xacro (robot description, xacro)
@@ -84,9 +84,11 @@
       <limit effort="12" velocity="1.0" lower="-2" upper="2"/>
     </joint>
+    <!-- The SDK returns wrist joint angles in physical order: axis 0, axis 1, axis 2.
+         On Lambda.07 axis 0 is parallel to world Z, so this visual chain uses Z/Y/X. -->
     <joint name="${robot_id}_roll" type="revolute">
       <origin rpy="0 0 0" xyz="0 0 0"/>
       <parent link="${robot_id}_z_link"/>
       <child link="${robot_id}_roll_link"/>
-      <axis xyz="1 0 0"/>
+      <axis xyz="0 0 1"/>
       <limit effort="0.4" velocity="10.0" lower="-3.14159265359" upper="3.14159265359"/>
     </joint>
@@ -102,5 +104,5 @@
       <parent link="${robot_id}_pitch_link"/>
       <child link="${robot_id}_yaw_link"/>
-      <axis xyz="0 0 1"/>
+      <axis xyz="1 0 0"/>
       <limit effort="0.4" velocity="10.0" lower="-3.14159265359" upper="3.14159265359"/>
     </joint>

Commit message: Align virtual clutch frame with handle Y axis

File: src/lambda07_bringup/urdf/lambda07.urdf.xacro (robot description, xacro)
@@ -116,5 +116,6 @@
       <parent link="${robot_id}_ee"/>
       <child link="${robot_id}_virtual_clutch_link"/>
-      <axis xyz="1 0 0"/>
+      <!-- Virtualized gripper/clutch state follows the handle-frame Y' side axis. -->
+      <axis xyz="0 1 0"/>
       <limit effort="12" velocity="1.0" lower="-0.05" upper="0.05"/>
     </joint>

Commit message: Document Lambda force status and clutch marker

File: src/lambda07_bringup/urdf/lambda07.urdf.xacro (robot description, xacro)
@@ -62,5 +62,13 @@
       </visual>
     </link>
-    <link name="${robot_id}_virtual_clutch_link"/>
+    <link name="${robot_id}_virtual_clutch_link">
+      <visual>
+        <origin xyz="0 0.035 0" rpy="1.57079632679 0 0"/>
+        <geometry>
+          <cylinder radius="0.004" length="0.07"/>
+        </geometry>
+        <material name="lambda07_axis_y"/>
+      </visual>
+    </link>
     <joint name="${robot_id}_x" type="prismatic">
       <origin rpy="0 0 0" xyz="0 0 0"/>
